Commit message: Added 'calibrated' table height and riser height.

File: godel_robots/abb/godel_irb4600/godel_irb4600_support/urdf/irb4600_workspace.xacro (robot description, xacro)
@@ -3,4 +3,5 @@
   <xacro:include filename="$(find abb_irb4600_support)/urdf/irb4600_60_205_macro.xacro"/>
   <xacro:include filename="$(find godel_irb4600_support)/urdf/pushcorp_macro.xacro"/>
+  <xacro:property name="riser_height" value=".72871"/>
   <link name="world_frame"/>
   <xacro:abb_irb4600_60_205 prefix=""/>
@@ -39,10 +40,10 @@
     <parent link="base_link"/>
     <child link="pedestal"/>
-    <origin xyz="0 0 -0.75" rpy="0 0 0"/>
+    <origin xyz="0 0 -${riser_height}" rpy="0 0 0"/>
   </joint>
   <joint name="base_link_to_table" type="fixed">
     <parent link="world_frame"/>
     <child link="table"/>
-    <origin xyz="0.75 -1.75 -0.75" rpy="0 0 0"/>
+    <origin xyz="1.40197 -1.45022 -0.56537" rpy="0 0 0"/>
   </joint>
   <joint name="tool0_to_tool1" type="fixed">

Commit message: Changed the referenced tool and added the calibrated tool frame for the keyence.

File: godel_robots/abb/godel_irb4600/godel_irb4600_support/urdf/irb4600_workspace.xacro (robot description, xacro)
@@ -6,6 +6,4 @@
   <link name="world_frame"/>
   <xacro:abb_irb4600_60_205 prefix=""/>
-  <!-- Todo: Tool definition -->
-  <link name="tool1"/>
   <link name="pedestal">
     <visual>
@@ -47,9 +45,4 @@
     <origin xyz="1.40197 -1.45022 -0.56537" rpy="0 0 0"/>
   </joint>
-  <joint name="tool0_to_tool1" type="fixed">
-    <parent link="tool0"/>
-    <child link="tool1"/>
-    <origin xyz="0 0 0" rpy="0 0 0"/>
-  </joint>
   <joint name="tool0_to_pushcorp" type="fixed">
     <parent link="tool0"/>

File: godel_robots/abb/godel_irb4600/godel_irb4600_support/urdf/pushcorp_macro.xacro (robot description, xacro)
@@ -26,10 +26,10 @@
     <parent link="tool_base_link"/>
     <child link="keyence_sensor_optical_frame"/>
-    <origin xyz="0.37157 0.41351 0.34975" rpy="3.14158331443 0.87266369146 2.35911267789"/>
+    <origin xyz="0.339156 0.384732 0.360953" rpy="-1.5615373368 0.882160345204 2.37121479211"/>
   </joint>
   <joint name="base_to_keyence_tcp_frame" type="fixed">
     <parent link="tool_base_link"/>
     <child link="keyence_tcp_frame"/>
-    <origin xyz="0.37157 0.41351 0.34975" rpy="1.57078698763 0.87266369146 2.35911267789"/>
+    <origin xyz="0.339156 0.384732 0.360953" rpy="1.58005531679 0.882160345204 2.37121479211"/>
   </joint>
   <!-- Blending Frame -->

Commit message: Added tool collision geometry and a 'no-go-zone'

File: godel_robots/abb/godel_irb4600/godel_irb4600_support/urdf/irb4600_workspace.xacro (robot description, xacro)
@@ -50,3 +50,16 @@
     <origin xyz="0 0 0" rpy="0 0 0"/>
   </joint>
+  <link name="no_go_zone">
+    <collision>
+      <origin xyz="0.4 0.75 0.05"/>
+      <geometry>
+        <box size="0.8 1.5 0.1"/>
+      </geometry>
+    </collision>
+  </link>
+  <joint name="table_to_no_go_zone" type="fixed">
+    <parent link="table"/>
+    <child link="no_go_zone"/>
+    <origin xyz="0 0 0.728" rpy="0 0 0"/>
+  </joint>
 </robot>

File: godel_robots/abb/godel_irb4600/godel_irb4600_support/urdf/pushcorp_macro.xacro (robot description, xacro)
@@ -50,3 +50,16 @@
     <origin xyz="0.10869 0.13329 0.24452" rpy="0.698133962102 -6.85595277301e-06 0.788324521691"/>
   </joint>
+  <!-- Special frame for collision avoidance -->
+  <link name="tcp_model">
+    <collision>
+      <geometry>
+        <mesh filename="package://godel_irb4600_support/meshes/collision/tcp.stl"/>
+      </geometry>
+    </collision>
+  </link>
+  <joint name="tcp_frame_to_model" type="fixed">
+    <parent link="tcp_frame"/>
+    <child link="tcp_model"/>
+    <origin xyz="0 0 0"/>
+  </joint>
 </robot>
