Commit message: Added nominal keyence mounting position

File: godel_robots/abb/godel_irb4600/godel_irb4600_support/urdf/pushcorp_macro.xacro (robot description, xacro)
@@ -26,10 +26,10 @@
     <parent link="tool_base_link"/>
     <child link="keyence_sensor_optical_frame"/>
-    <origin xyz="0 0 0" rpy="0 0 0"/>
+    <origin xyz="0.37157 0.41351 0.34975" rpy="3.14158331443 0.87266369146 2.35911267789"/>
   </joint>
   <joint name="base_to_keyence_tcp_frame" type="fixed">
     <parent link="tool_base_link"/>
     <child link="keyence_tcp_frame"/>
-    <origin xyz="0 0 0" rpy="0 0 0"/>
+    <origin xyz="0.37157 0.41351 0.34975" rpy="1.57078698763 0.87266369146 2.35911267789"/>
   </joint>
   <!-- Blending Frame -->

Commit message: Updated grinding tcp

File: godel_robots/abb/godel_irb4600/godel_irb4600_support/urdf/pushcorp_macro.xacro (robot description, xacro)
@@ -37,5 +37,5 @@
     <parent link="tool_base_link"/>
     <child link="tcp_frame"/>
-    <origin xyz="-0.053385 0.053384 0.527808" rpy="3.3621683182e-12 0.872664625459 2.35619448997"/>
+    <origin xyz="-0.061890167647 0.064044258542 0.54800788851" rpy="-0.00320361244442 0.880669021029 2.32406931184"/>
   </joint>
   <!-- Macro-Scanner Frames -->

Commit message: Added a nominal transform and tilted the keyence a little to make the calibration work out right.

File: godel_robots/abb/godel_irb4600/godel_irb4600_support/urdf/pushcorp_macro.xacro (robot description, xacro)
@@ -24,7 +24,7 @@
   <!-- Laser scanner joints -->
   <joint name="base_to_keyence_optical_frame" type="fixed">
-    <parent link="tool_base_link"/>
+    <parent link="keyence_optical_base"/>
     <child link="keyence_sensor_optical_frame"/>
-    <origin xyz="0.339156 0.384732 0.360953" rpy="-1.5615373368 0.882160345204 2.37121479211"/>
+    <origin xyz="0 0 0" rpy="0 0.015 0"/>
   </joint>
   <joint name="base_to_keyence_tcp_frame" type="fixed">
@@ -32,4 +32,10 @@
     <child link="keyence_tcp_frame"/>
     <origin xyz="0.339156 0.384732 0.360953" rpy="1.58005531679 0.882160345204 2.37121479211"/>
+  </joint>
+  <link name="keyence_optical_base"/>
+  <joint name="base_to_keyence_optical_base" type="fixed">
+    <parent link="tool_base_link"/>
+    <child link="keyence_optical_base"/>
+    <origin xyz="0.339156 0.384732 0.360953" rpy="-1.5615373368 0.882160345204 2.37121479211"/>
   </joint>
   <!-- Blending Frame -->
